File: WeMos-Matrix-Shield-DMA.brd (EAGLE design)
At the start: 50.9 x 49.5 mm, 23 parts, among them J3 TWIG-2.0-DIP, U1 LDR, X1 5202-02-N-02

Commit message: bump to v1.8a
Parts:
- added C1: 100uf, Seeed-Capacitor:PC-D5.3MM
- added C2, C3: (no value), _c2h:0805-CAP-LARGEPADS
- moved J3 3.81 mm to (23.5, 30.0)
Connections:
- net 3V3: now also C1.+, C2.1, C3.1
- net GND: now also C1.-, C2.2, C3.2
Routing:
- net 3V3: track 37.2 -> 43.2 mm, vias 1 -> 0
- net SDA: track 69.3 -> 73.1 mm
- net SCL: track 59.6 -> 63.4 mm
- net VCC: track 38.4 -> 39.7 mm
- net GND: vias 22 -> 23
Other:
- board text added: "ESP32 Matrix Shield DMA V1.8a"
- board text removed: "ESP32 Matrix Shield DMA V1.8"

Commit message: Updated to V1.9
Parts:
- removed J4: (no value), SparkFun-Connectors:1X04_LOCK
- added J1: I2C, _c2h:1X04_LOCK_HOLE
- added P2: PADSMALL, _c2h:PAD-SMALL
- J2: value TWIG-2.0-DIP -> GROOVE
- moved JP4 17.1 mm to (66.0, 27.2)
- moved C2 12.0 mm to (35.1, 34.2), turned to 180 degrees
- moved C3 9.54 mm to (35.1, 36.3), turned to 180 degrees
- moved R3 9.40 mm to (19.8, 45.1)
- moved R1 8.54 mm to (33.9, 55.6), turned to 270 degrees
- moved R4 4.70 mm to (19.8, 47.6)
- moved X2 3.81 mm to (64.8, 37.5)
- moved U$2 2.54 mm to (31.1, 45.7)
- moved U$4 2.54 mm to (28.6, 45.7)
- moved U$5 2.54 mm to (56.5, 45.7)
- moved U$6 2.54 mm to (54.0, 45.7)
- moved C1 0.90 mm to (23.7, 38.5)
- moved D3 0.63 mm to (59.1, 29.8), turned to 270 degrees
- moved X1 0.38 mm to (62.5, 17.0)
- renumbered J3 to J2
Connections:
- new net IO10: U$2.10
- net GND: now also J1.2; no longer J4.2
- net IO0: now also JP6.2
- net IO2: no longer B1.BUTTON
- net IO32: now also B1.BUTTON; no longer JP5.2
- net IO33: now also JP5.2; no longer JP6.2
- net IO34: now also P2.1
- net SCL: now also J1.3; no longer J4.3
- net SDA: now also J1.4; no longer J4.4
- net VCC: now also J1.1; no longer J4.1
Routing:
- net IO32: track 13.1 -> 47.6 mm
- net IO2: track 31.7 -> 0.00 mm
- net IO0: track 0.00 -> 15.3 mm
- net 5V-EXT: track 78.8 -> 68.9 mm
- net SDA: track 73.1 -> 63.4 mm, vias 0 -> 1
- net SCL: track 63.4 -> 54.4 mm
- net 3V3: track 43.2 -> 51.2 mm
- net IO34: track 0.00 -> 6.38 mm
- net GND: track 22.3 -> 17.0 mm, vias 23 -> 33
- net IO19: track 23.3 -> 18.6 mm
- net IO33: track 34.9 -> 39.6 mm
- net A0: track 8.57 -> 12.5 mm
- net IO25: track 18.3 -> 22.1 mm
- net IO4: track 21.9 -> 25.5 mm
- net IO12: track 14.7 -> 18.2 mm
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Other:
- outline, holes or cut-outs redrawn
- board text added: "0"
- board text added: "ESP32 Matrix Shield DMA V1.9"
- board text added: "IO34"
- board text added: "T9 (IO32)"
- board text removed: "32"
- board text removed: "ESP32 Matrix Shield DMA V1.8a"
- board text removed: "IO2"
- board text removed: "Touch"
