File: WeMos-Matrix-Shield-DMA.sch (EAGLE design)
At the start: 21 parts, among them J3 TWIG-2.0-DIP, U1 LDR, X1 5202-02-N-02

Commit message: bump to v1.8a
Parts:
- added C1: 100uf, Seeed-Capacitor:DIP-ALUMINUM-47UF-16V(D5-H7MM)
- added C2, C3: (no value), _c2h:CAP0805-CAP-LARGEPADS
Connections:
- net 3V3: now also C1.+, C2.1, C3.1
- net GND: now also C1.-, C2.2, C3.2
Other:
- note added: "C1, C2, C3 are footprint to add capacitor to poor 3.3V VOut of esp32 on board regulator. This one is not output filtered enough resulting sometimes with brownout reset loop. Now you can plug radial or 1 (or 2) SMD 0805 in //"
- moved on the sheet: U$5, U$6

Commit message: Updated to V1.9
Parts:
- removed J4: (no value), SparkFun-Connectors:CONN_04LOCK
- added J1: I2C, _c2h:CON_HEADER_1X04SMALLHOLE
- added P2: PADSMALL, _c2h:PADSMALL
- J2: value TWIG-2.0-DIP -> GROOVE
- renumbered J3 to J2
Connections:
- new net IO10: U$2.10
- net GND: now also J1.2; no longer J4.2
- net IO0: now also JP6.2
- net IO2: no longer B1.BUTTON
- net IO32: now also B1.BUTTON; no longer JP5.2
- net IO33: now also JP5.2; no longer JP6.2
- net IO34: now also P2.1
- net SCL: now also J1.3; no longer J4.3
- net SDA: now also J1.4; no longer J4.4
- net VCC: now also J1.1; no longer J4.1
Other:
- note added: "LED"
- moved on the sheet: R1, U1
